File: main-robot.brd (EAGLE design)
At the start: 100 x 100 mm, 114 parts, among them CON1 AX12, CON2 AX12, SW1 SWITCH-SPDT-H, SW2 PUSH-BUTTON436331045822, SW3 PUSH-BUTTON, SW4 PUSH-BUTTON, SW5 PUSH-BUTTON436331045822, SW6 PUSH-BUTTON436331045822, SW7 PUSH-BUTTON436331045822, U1 TEENSY_3.5_DIL+4

Commit message: brd: add more GND vias
Routing:
- net GND: vias 17 -> 55
Changed lines of the file:
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@@
 <via x="65.8" y="66.5" extent="1-16" drill="0.35" shape="octagon"/>
 <via x="57.5" y="66.6" extent="1-16" drill="0.35" shape="octagon"/>
+<via x="8.2" y="37.4" extent="1-16" drill="0.35" shape="octagon"/>
+<via x="9.2" y="37.7" extent="1-16" drill="0.35" shape="octagon"/>
+<via x="9.2" y="35.8" extent="1-16" drill="0.35" shape="octagon"/>
+<via x="8.5" y="39.8" extent="1-16" drill="0.35" shape="octagon"/>
+<via x="9.2" y="40.5" extent="1-16" drill="0.35" shape="octagon"/>
+<via x="8.6" y="45.1" extent="1-16" drill="0.35" shape="octagon"/>
+<via x="11" y="45.1" extent="1-16" drill="0.35" shape="octagon"/>
+<via x="12.7" y="45.6" extent="1-16" drill="0.35" shape="octagon"/>
+<via x="20.3" y="45.6" extent="1-16" drill="0.35" shape="octagon"/>
+<via x="20.3" y="49.7" extent="1-16" drill="0.35" shape="octagon"/>
+<via x="15.2" y="49.9" extent="1-16" drill="0.35" shape="octagon"/>
+<via x="20.3" y="51.8" extent="1-16" drill="0.35" shape="octagon"/>
+<via x="15.2" y="52" extent="1-16" drill="0.35" shape="octagon"/>
+<via x="27.9" y="45.3" extent="1-16" drill="0.35" shape="octagon"/>
+<via x="33" y="45.3" extent="1-16" drill="0.35" shape="octagon"/>
+<via x="27.9" y="49.7" extent="1-16" drill="0.35" shape="octagon"/>
+<via x="33" y="49.7" extent="1-16" drill="0.35" shape="octagon"/>
+<via x="27.9" y="51.7" extent="1-16" drill="0.35" shape="octagon"/>
+<via x="33" y="51.7" extent="1-16" drill="0.35" shape="octagon"/>
+<via x="14.1" y="75.1" extent="1-16" drill="0.35" shape="octagon"/>
+<via x="16.1" y="75.1" extent="1-16" drill="0.35" shape="octagon"/>
+<via x="23.6" y="72.6" extent="1-16" drill="0.35" shape="octagon"/>
+<via x="57.1" y="52.6" extent="1-16" drill="0.35" shape="octagon"/>
+<via x="58.7" y="52.6" extent="1-16" drill="0.35" shape="octagon"/>
+<via x="69" y="96.5" extent="1-16" drill="0.35" shape="octagon"/>
+<via x="68.1" y="96.5" extent="1-16" drill="0.35" shape="octagon"/>
+<via x="69.9" y="96.5" extent="1-16" drill="0.35" shape="octagon"/>
+<via x="69" y="87.5" extent="1-16" drill="0.35" shape="octagon"/>
+<via x="68.1" y="87.5" extent="1-16" drill="0.35" shape="octagon"/>
+<via x="69.9" y="87.5" extent="1-16" drill="0.35" shape="octagon"/>
+<via x="74.6" y="90.6" extent="1-16" drill="0.35" shape="octagon"/>
+<via x="81.1" y="82.3" extent="1-16" drill="0.35" shape="octagon"/>
+<via x="81.1" y="78.3" extent="1-16" drill="0.35" shape="octagon"/>
+<via x="12.6" y="27.1" extent="1-16" drill="0.35" shape="octagon"/>
+<via x="9" y="31" extent="1-16" drill="0.35" shape="octagon"/>
+<via x="14.7" y="35.9" extent="1-16" drill="0.35" shape="octagon"/>
+<via x="16.3" y="35.9" extent="1-16" drill="0.35" shape="octagon"/>
+<via x="13.1" y="31.6" extent="1-16" drill="0.35" shape="octagon"/>
 </signal>
 <signal name="N$1">
