File: main-robot.brd (EAGLE design)
At the start: 100 x 100 mm, 114 parts, among them CON1 AX12, CON2 AX12, SW1 SWITCH-SPDT-H, SW2 PUSH-BUTTON436331045822, SW3 PUSH-BUTTON, SW4 PUSH-BUTTON, SW5 PUSH-BUTTON436331045822, SW6 PUSH-BUTTON436331045822, SW7 PUSH-BUTTON436331045822, U1 TEENSY_3.5_DIL+4

Commit message: add connector for rpi with 3D model
Parts:
- SV1: device con-lsta:FE20-2 -> con-raspberry-pi:FE20-2
Changed lines of the file:
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@@
 </layers>
 <board>
-<fusionsync huburn="a.cGVyc29uYWw6dWUyYjVjZTIy" projecturn="a.cGVyc29uYWw6dWUyYjVjZTIyIzIwMTkwOTI4MjIwMDY0MjI2" f3durn="urn:adsk.wipprod:dm.lineage:Tw-aWBHUQ9-QpGxy24Xodg" pcbguid="a969bc88-2eb4-46df-86c6-0b31fed4e920" lastpulledtime="" lastsyncedchangeguid="5a5d8461-ca6c-1b82-456d-72ecfe42a188"/>
+<fusionsync huburn="a.cGVyc29uYWw6dWUyYjVjZTIy" projecturn="a.cGVyc29uYWw6dWUyYjVjZTIyIzIwMTkwOTI4MjIwMDY0MjI2" f3durn="urn:adsk.wipprod:dm.lineage:Tw-aWBHUQ9-QpGxy24Xodg" pcbguid="a969bc88-2eb4-46df-86c6-0b31fed4e920" lastpulledtime="" lastsyncedchangeguid="f3dc9b47-4484-8e1f-c7ba-72fd607cfdf6"/>
 <plain>
 <wire x1="0" y1="95.4848625" x2="0" y2="49.8050625" width="0.001" layer="20" locked="yes"/>
@@
 <attribute name="RS" value="517-6966" x="53.77" y="-10.59" size="1.778" layer="28" rot="MR270" display="off"/>
 </element>
-<element name="SV1" library="con-lsta" library_urn="urn:adsk.eagle:library:161" package="FE20-2" package3d_urn="urn:adsk.eagle:package:8184/1" value="RPI" x="25.4" y="47.6650625" locked="yes" smashed="yes">
-<attribute name="MF" value="" x="25.4" y="47.6650625" locked="yes" size="1.778" layer="27" display="off"/>
-<attribute name="MPN" value="" x="25.4" y="47.6650625" locked="yes" size="1.778" layer="27" display="off"/>
-<attribute name="OC_FARNELL" value="unknown" x="25.4" y="47.6650625" locked="yes" size="1.778" layer="27" display="off"/>
-<attribute name="OC_NEWARK" value="unknown" x="25.4" y="47.6650625" locked="yes" size="1.778" layer="27" display="off"/>
-<attribute name="POPULARITY" value="0" x="25.4" y="47.6650625" locked="yes" size="1.778" layer="27" display="off"/>
+<element name="SV1" library="con-raspberry-pi" library_urn="urn:adsk.eagle:library:16832158" package="FE20-2" package3d_urn="urn:adsk.eagle:package:16832194/2" value="RPI" x="25.4" y="47.6650625" locked="yes" smashed="yes">
+<attribute name="MANUFACTURER" value="Samtec" x="25.4" y="47.6650625" size="1.778" layer="27" display="off"/>
+<attribute name="MOUSER" value="200-ESW12048GD" x="25.4" y="47.6650625" size="1.778" layer="27" display="off"/>
+<attribute name="REF" value="ESW-120-48-G-D" x="25.4" y="47.6650625" size="1.778" layer="27" display="off"/>
 <attribute name="VALUE" x="0" y="42.9660625" locked="yes" size="1.27" layer="27" ratio="10"/>
 </element>

Commit message: change Flag connector
Parts:
- added C12, C13: 100nF, resistor:C0805
- added JMP2: 0R-JUMPA, jump-0r-smd:A0R-JMP
- FLAG: value GENERIC-4PIN53253 -> JST-05TOP; device con-molex-dynamixel:53253-0470 -> con-jst-gh:BM05B-GHS
- moved FLAG 1.00 mm to (61.0, 94.0)
Connections:
- new net N$22: JMP2.2, LEDS.3, LEDS.4
- net +5V/1: now also JMP2.3; no longer LEDS.3, LEDS.4
- net EXT_+5V: now also JMP2.1
- net FLAG_GPIO1: now also C12.1
- net FLAG_GPIO2: now also C13.1
- net GND: now also C12.2, C13.2, FLAG.1
- net N$5: now also FLAG.5; no longer FLAG.1
- net N$6: now also FLAG.4; no longer FLAG.2
- net N$8: now also FLAG.2; no longer FLAG.4
Routing:
- net N$22: track 0.00 -> 54.6 mm, vias 0 -> 1
- net +5V/1: track 264.2 -> 258.6 mm
- net N$8: track 8.54 -> 11.6 mm, vias 0 -> 1
- net EXT_+5V: track 54.8 -> 57.0 mm
- net N$7: track 12.2 -> 14.5 mm, vias 0 -> 1
- net FLAG_GPIO1: track 86.1 -> 87.9 mm
- net N$5: track 10.3 -> 8.57 mm, vias 0 -> 1
- net FLAG_GPIO2: track 88.0 -> 89.5 mm
- net N$6: track 13.9 -> 13.7 mm, vias 0 -> 1
- net GND: vias 55 -> 58
Other:
- board text added: "5V"
- board text added: "EXT_5V"
- board text added: "LEDS"
- board text removed: "+5V"
