File: main-robot.sch (EAGLE design)
At the start: 75 parts, among them CON1 AX12, CON2 AX12, SW1 SWITCH-SPDT-H, SW2 PUSH-BUTTON436331045822, SW3 PUSH-BUTTON, SW4 PUSH-BUTTON, SW5 PUSH-BUTTON436331045822, SW6 PUSH-BUTTON436331045822, SW7 PUSH-BUTTON436331045822, U1 TEENSY_3.5_DIL+4

Commit message: add connector for rpi with 3D model
Parts:
- SV1: device con-lsta:FE20-2 -> con-raspberry-pi:FE20-2
Changed lines of the file:
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@@
 <part name="GND4" library="supply1" library_urn="urn:adsk.eagle:library:371" deviceset="GND" device=""/>
 <part name="GND5" library="supply1" library_urn="urn:adsk.eagle:library:371" deviceset="GND" device=""/>
-<part name="SV1" library="con-lsta" library_urn="urn:adsk.eagle:library:161" deviceset="FE20-2" device="" package3d_urn="urn:adsk.eagle:package:8184/1" value="RPI"/>
+<part name="SV1" library="con-raspberry-pi" library_urn="urn:adsk.eagle:library:16832158" deviceset="FE20-2" device="" package3d_urn="urn:adsk.eagle:package:16832194/2" value="RPI"/>
 <part name="LIPO+" library="testpad" library_urn="urn:adsk.eagle:library:385" deviceset="TP" device="PAD1-20Y" package3d_urn="urn:adsk.eagle:package:27951/1"/>
 <part name="LIPO-" library="testpad" library_urn="urn:adsk.eagle:library:385" deviceset="TP" device="PAD1-20Y" package3d_urn="urn:adsk.eagle:package:27951/1"/>

Commit message: change Flag connector
Parts:
- added C12, C13: 100nF, resistor:C-EUC0805
- added JMP2: 0R-JUMPA, jump-0r-smd:0R-JUMPA
- FLAG: value GENERIC-4PIN53253 -> JST-05TOP; device con-molex-dynamixel:GENERIC-4PIN53253 -> con-jst-gh:JST-05TOP
Connections:
- new net N$22: JMP2-0R.2, LEDS.3, LEDS.4
- net +5V/1: now also JMP2-0R.3; no longer LEDS.3, LEDS.4
- net EXT_+5V: now also JMP2-0R.1
- net FLAG_GPIO1: now also C12.1
- net FLAG_GPIO2: now also C13.1
- net GND: now also C12.2, C13.2, FLAG.1
- net N$5: now also FLAG.5; no longer FLAG.1
- net N$6: now also FLAG.4; no longer FLAG.2
- net N$8: now also FLAG.2; no longer FLAG.4
Other:
- moved on the sheet: R1, R2
